File: nixie.kicad_pcb (KiCad board)
At the start: 4 copper layers, 182.5 x 65.2 mm, 55 parts, among them IC1 SN74141, IC2 SN74141, IC3 SN74141, IC4 SN74141, IC5 MCP23017-E_SO, IC6 DS3231M+TRL, IC7 SN74141, IC8 SN74141, IC9 L7805CD2T-TR, J2 M20-9990646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

Commit message: Changes to schematic
Parts:
- removed J2: M20-9990646, footprints:HDRV6W64P0X254_1X6_1524X254X864P
- U$1: moved to F.Cu
- moved U$1 3.31 mm to (100.8, 127.1)

Commit message: Started routing
Parts:
- removed C12: 100nf, nixie:C0805
- added J1: M20-9990446, footprints:HDRV4W64P0X254_1X4_1016X254X889P, F.Cu at (70.0, 119.5)
- added R11: 10k, nixie:R0805, F.Cu at (175.5, 127.9)
- C10, C11, C6, IC9: moved to B.Cu
- moved C6 38.5 mm to (118.9, 133.0), turned to 180 degrees
- moved R5 31.7 mm to (145.2, 122.0)
- moved IC6 31.7 mm to (135.7, 126.8)
- moved R6 31.7 mm to (145.2, 124.0)
- moved C5 30.3 mm to (136.3, 122.7)
- moved C7 24.4 mm to (167.0, 126.4)
- moved R10 22.6 mm to (157.9, 128.2)
- moved R9 22.6 mm to (157.9, 130.4)
- moved IC5 22.5 mm to (166.7, 123.4)
- moved C10 11.5 mm to (219.2, 127.0)
- moved C11 11.4 mm to (219.5, 121.9), turned to -90 degrees
- moved IC9 10.3 mm to (230.1, 123.5)
- moved J3 2.54 mm to (210.0, 137.5), turned to 0 degrees
- moved J4 1.97 mm to (225.0, 137.6), turned to 0 degrees
- moved S1 1.49 mm to (133.4, 138.6)
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Connections:
- IC5 pad 1: /A1 -> /A4
- IC5 pad 18: unconnected-(IC5-~{RESET}-Pad18) -> /RST
- IC5 pad 2: /B1 -> /D4
- IC5 pad 21: /D4 -> /C6
- IC5 pad 22: /C4 -> /B6
- IC5 pad 23: /B4 -> /D6
- IC5 pad 24: /A4 -> /A6
- IC5 pad 25: /D3 -> /C5
- IC5 pad 26: /C3 -> /B5
- IC5 pad 27: /B3 -> /D5
- IC5 pad 28: /A3 -> /A5
- IC5 pad 3: /C1 -> /B4
- IC5 pad 4: /D1 -> /C4
- IC5 pad 5: /A2 -> /C3
- IC5 pad 6: /B2 -> /B3
- IC5 pad 7: /C2 -> /D3
- IC5 pad 8: /D2 -> /A3
- IC6 pad 15: /SDA -> /SDA1
- IC6 pad 16: /SCL -> /SCL1
- R10 pad 2: +5V -> +3V3
- R5 pad 1: /SCL -> /SCL1
- R5 pad 2: +5V -> +3V3
- R6 pad 1: /SDA -> /SDA1
- R6 pad 2: +5V -> +3V3
- R9 pad 2: +5V -> +3V3
- U$1 pad GP0: /SDA -> /RX
- U$1 pad GP1: /SCL -> /TX
- U$1 pad GP10: /C5 -> /C1
- U$1 pad GP11: /D5 -> /B1
- U$1 pad GP12: /A6 -> /D1
- U$1 pad GP13: /B6 -> /A1
- U$1 pad GP14: /C6 -> /SDA1
- U$1 pad GP15: /D6 -> /SCL1
- U$1 pad GP16: /S1 -> /S6
- U$1 pad GP17: /S2 -> /S5
- U$1 pad GP18: /S3 -> /S4
- U$1 pad GP19: /S4 -> /S3
- U$1 pad GP2: /SWCLK -> /RST
- U$1 pad GP20: /S5 -> /S2
- U$1 pad GP21: /S6 -> /S1
- U$1 pad GP3: /SWDIO -> unconnected-(U$1-PadGP3)
- U$1 pad GP4: /RX -> /C2
- U$1 pad GP5: /TX -> /B2
- U$1 pad GP6: /SDA1 -> /D2
- U$1 pad GP7: /SCL1 -> /A2
- U$1 pad GP8: /A5 -> unconnected-(U$1-PadGP8)
- U$1 pad GP9: /B5 -> unconnected-(U$1-PadGP9)
Routing:
- net +5V: track 0.00 -> 334.8 mm, vias 0 -> 3
- net VCC: track 0.00 -> 224.2 mm
- net +3V3: track 0.00 -> 223.6 mm
- net /S6: track 0.00 -> 107.4 mm, vias 0 -> 1
- net /SDA1: track 0.00 -> 106.9 mm, vias 0 -> 4
- net /SCL1: track 0.00 -> 104.4 mm, vias 0 -> 2
- net /S5: track 0.00 -> 94.4 mm, vias 0 -> 1
- net /S4: track 0.00 -> 79.7 mm, vias 0 -> 1
- net /C6: track 0.00 -> 73.5 mm
- net /S3: track 0.00 -> 70.4 mm
- net /B6: track 0.00 -> 69.7 mm
- net /RST: track 0.00 -> 69.4 mm, vias 0 -> 1
- net Net-(IC6-VBAT): track 0.00 -> 64.6 mm, vias 0 -> 1
- net /D6: track 0.00 -> 63.5 mm
- net /A6: track 0.00 -> 60.5 mm
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
Commit message: made minor changes to routing
Parts:
- moved U$2 125.9 mm to (253.1, 107.3)
- moved G*** 80.6 mm to (153.7, 112.0)
- moved C6 2.60 mm to (121.5, 133.0)
- moved C5 2.16 mm to (134.2, 122.5)
- moved C7 1.50 mm to (165.5, 126.3)
- renumbered U$1 to Pi1
Routing:
- net +5V: track 334.8 -> 327.9 mm
- net /N27: track 41.6 -> 48.3 mm, vias 4 -> 1
- net /N47: track 37.9 -> 42.7 mm, vias 2 -> 0
- net /N37: track 37.5 -> 42.2 mm, vias 2 -> 0
- net /N26: track 38.1 -> 42.5 mm, vias 1 -> 0
- net /N57: track 38.4 -> 42.3 mm, vias 2 -> 0
- net GND: track 55.2 -> 58.0 mm, vias 12 -> 11
- net /S6: track 107.4 -> 105.5 mm
- net /N14: track 24.6 -> 25.9 mm
- net /D6: track 63.5 -> 64.7 mm
- net /S5: track 94.4 -> 93.4 mm
- net /N22: track 27.0 -> 27.9 mm
- net /SDA1: track 106.9 -> 106.0 mm, vias 4 -> 3
- net /D5: track 35.5 -> 36.3 mm
- net +3V3: track 223.6 -> 224.4 mm
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Other:
- board text added: "3V3"
- board text added: "H+"
- board text added: "H-"
- board text added: "M+"
- board text added: "M-"
- board text added: "RX"
- board text added: "S+"
- board text added: "S-"
- board text added: "SWCLK"
- board text added: "SWDIO"
- board text added: "TX"
- board text removed: "DANGER! 170V"

Commit message: added vias, made small routing adjustments
Parts:
- removed U$3: BIGPP, nixie:BIGPP
- moved U$2 75.1 mm to (179.8, 90.9)
- moved G*** 1.43 mm to (155.1, 111.7)
Routing:
- net GND: vias 11 -> 197
Other:
- board text added: "JLCJLCJLCJLC"
- board text added: "Warning! 170V"

Commit message: added reset line for clock
Parts:
- renumbered Pi1 to P1
Connections:
- net /RST renamed /RSTIO
- IC6 pad 4: unconnected-(IC6-~{RST}-Pad4) -> /RSTC
- P1 pad GP3: unconnected-(U$1-PadGP3) -> /RSTC
Routing:
- net /RSTC: track 0.00 -> 28.9 mm
- net GND: vias 197 -> 216
